File: STamps-01/schematic-1.sch (EAGLE design)
At the start: 114 parts, among them IC2 LT1763CS8-3.3, Q1 BSH105, Q2 BSH105, Q5 BSH105, T1 PSMN7R0-30YL, T2 PSMN7R0-30YL, T5 PSMN7R0-30YL

Commit message: Added PDF Files
PDF Files for Eagle schematics, nothing new for KiCad ATM
Connections:
- removed net N$9: U$1.BOOT0
- new net SPI_CS1: U$1.PB12
- new net SPI_CS2: U$1.PC6
- net BOOT0: now also U$1.BOOT0
- net E0_DIR: now also U$1.PA1
- net E0_EN: now also U$1.PC3
- net E0_STEP: now also U$1.PA0-WKUP
- net I2C_SCL: now also U$1.PB6; no longer U$1.PB10
- net I2C_SDA: now also U$1.PB7; no longer U$1.PB11
- net NRST: now also U$1.NRST
- net SPI_CS: no longer U$1.PB12
- net SWCLK: now also U$1.PA14
- net SWDIO: now also U$1.PA13
- net SWO: now also U$1.PA15
- net T0: now also U$1.PC5
- net T1: now also U$1.PB0
- net T2: now also U$1.PB1
- net X-MAX: now also U$1.PA4
- net X-MIN: now also U$1.PA2
- net X_DIR: now also U$1.PB4
- net X_EN: now also U$1.PD2
- net X_STEP: now also U$1.PB3
- net Y-MAX: now also U$1.PA6
- net Y-MIN: now also U$1.PA5
- net Y_DIR: now also U$1.PB9
- net Y_EN: now also U$1.PB5
- net Y_STEP: now also U$1.PB8
- net Z-MAX: now also U$1.PC4
- net Z-MIN: now also U$1.PA7
- net Z_DIR: now also U$1.PC2
- net Z_EN: now also U$1.PC0
- net Z_STEP: now also U$1.PC1
Other:
- note added: "TODO: -12/24V Input ->Heatbed ->Stepper/Electronics/Fan -Search SMD Car Fuse Holder"
- note removed: "TODO: -12/24V Input ->Heatbed ->Stepper/Electronics/Fan -Search SMD Car Fuse Holder -Pinout ->SmartLCD Adapter Compatible ->SDramps Compatible -> Rest EXTRA -MCU Crystal 8Mhz"
- moved on the sheet: C7, C8, CN1, D7, JS10, JS11, JS12, JS7, JS8, JS9, R30, R31
