File: STaps-01 KiCad/STaps-01.sch (KiCad schematic (older format))
At the start: 5 parts

Commit message: changes to kicad
Parts:
- removed C?: CAP, symbol CAP
- removed U? (x4): POLOLU_A4988, symbol POLOLU_A4988
- added C? (x4): 0.1uF, symbol C
- added C?: 1uF, symbol C
- added C?: 10nF, symbol C
- added C?: 4.7uF, symbol C
- added C? (x2): 100uF, symbol CP1_Small
- added P? (x2): 2X3, symbol CONN_02X03
- added P? (x2): CONN_02X04, symbol CONN_02X04
- added P? (x2): SCREW-TERMINAL, symbol CONN_01X04
- added R? (x2): R, symbol R
- added U?: STM32F103RC, LQFP64, symbol STM32F103RC
- added U? (x2): POLOLU_A4988, symbol POLOLU_A4988
- added X?: 8MHz, symbol CRYSTAL_SMD
Connections:
- new net: U?.5 (PD0/OSC_IN), X?.1
- new net: U?.6 (PD1/OSC_OUT), X?.2
- new net: P?.5 (P5), R?.1, U?.10 (MS1) (x2)
- new net: P?.3 (P3), U?.11 (MS2) (x2)
- new net: P?.1 (P1), U?.12 (MS3) (x2)
- new net: U?.13 (RST), U?.14 (SLP) (x2)
- new net: P?.2 (P2), U?.3 (IB) (x2)
- new net: P?.4 (P4), U?.4 (1A) (x2)
- new net: P?.6 (P6), U?.5 (2A) (x2)
- new net: P?.8 (P8), U?.6 (2B) (x2)
- new net: P?.1 (P1), P?.4 (P4) (x2)
- new net: P?.3 (P3), P?.3 (P3) (x2)
- new net: P?.2 (P2), P?.5 (P5) (x2)
- new net: P?.1 (P1), P?.7 (P7) (x2)
- new net +12V: C?.1, C?.1, U?.8 (VMOT), U?.8 (VMOT)
- new net +3V3: C?.1, C?.1, C?.1, C?.1, C?.1, C?.1, C?.1, P?.2 (P2), P?.2 (P2), P?.4 (P4), P?.4 (P4), P?.6 (P6), P?.6 (P6), U?.13 (VDDA), U?.19 (VDD), U?.2 (VDD), U?.2 (VDD), U?.32 (VDD), U?.48 (VDD), U?.64 (VDD)
- new net BL-RX: U?.52 (PC11/UART4_RX/SDIO_D3)
- new net BL-TX: U?.51 (PC10/UART4_TX/SDIO_D2)
- new net BOOT0: U?.60 (BOOT0)
- new net BOOT1: U?.28 (BOOT1/PB2)
- new net E0: U?.39 (PC8/TIM8_CH3/SDIO_D0)
- new net E0-DIR: U?.15 (USART2_RTS/ADC123_IN1/TIM5_CH2/TIM2_CH2/PA1)
- new net E0-EN: U?.11 (PC3/ADC123_IN13)
- new net E0-STEP: U?.14 (WKUP/USART2_CTS/ADC123_IN0/TIM2_CH1_ETR/TIM5_CH1/TIM8_ETR/PA0)
- new net EXTRA0: U?.38 (PC7/I2S3_MCK/TIM8_CH2/SDIO_D7)
- new net GND: C?.2, C?.2, C?.2, C?.2, C?.2, C?.2, C?.2, C?.2, C?.2, R?.2, R?.2, U?.1 (GND), U?.1 (GND), U?.12 (VSSA), U?.18 (VSS), U?.31 (VSS), U?.47 (VSS), U?.63 (VSS), U?.7 (GND), U?.7 (GND)
- new net HEATBED: U?.40 (PC9/TIM8_CH4/SDIO_D1)
- new net I2C-SCL: U?.58 (I2C1_SCL/TIM4_CH1/PB6)
- new net I2C-SDA: U?.59 (I2C1_SDA/TIM4_CH2/PB7)
- new net NRST: U?.7 (~NRST)
- new net SPI-CS1: U?.33 (SPI2_NSS/I2S2_WS/I2C2_SMBA/USART3_CK/TIM1_BKIN/PB12)
- new net SPI-CS2: U?.37 (PC6/I2S2_MCK/TIM8_CH1/SDIO_D6)
- new net SPI-MISO: U?.35 (SPI2_MISO/TIM1_CH2N/USART3_RTS/PB14)
- new net SPI-MOSI: U?.36 (SPI2_MOSI/I2S2_SD/TIM1_CH3N/PB15)
- new net SPI-SCK: U?.34 (SPI2_SCK/I2S2_CK/USART3_CTS/TIM1_CH1N/PB13)
- new net SWCLK: U?.49 (JTCK/SWCLK/PA14)
- new net SWDIO: U?.46 (JTMS/SWDIO/PA13)
- new net SWO: U?.50 (JTDI/SPI3_NSS/I2S3_WS/PA15)
- new net T0: U?.25 (PC5/ADC12_IN15)
- new net T1: U?.26 (ADC12_IN8/TIM3_CH3/TIM8_CH2N/PB0)
- new net T2: U?.27 (ADC12_IN9/TIM3_CH4/TIM8_CH3N/PB1)
- new net UART1-RX: U?.42 (USART1_TX/TIM1_CH2/PA9)
- new net UART1-TX: U?.43 (USART1_RX/TIM1_CH3/PA10)
- new net USBDM: U?.44 (USART1_CTS/USBDM/CAN_RX/TIM1_CH4/PA11)
- new net USBDP: U?.45 (USART1_RTS/USBDP/CAN_TX/TIM1_ETR/PA11)
- new net X-DIR: U?.56 (NJTRST/SPI3_MISO/PB4)
- new net X-EN: U?.54 (PD2/TIM3_ETR/UART5_RX/SDIO_CMD)
- new net X-MAX: U?.20 (SPI1_NSS/USART2_CK/DAC_OUT1/ADC12_IN4/PA4)
- new net X-MIN: U?.16 (USART2_TX/TIM5_CH3/ADC123_IN2/TIM2_CH3/PA2)
- new net X-STEP: U?.55 (JTDO/SPI3_SCK/I2S3_CK/PB3)
- new net Y-DIR: U?.62 (TIM4_CH4/SDIO_D5/PB9)
- new net Y-EN: U?.57 (I2C1_SMBA/SPI3_MOSI/I2S3_CD/PB5)
- new net Y-MAX: U?.22 (SPI1_MISO/TIM8_BKIN/ADC12_IN6/TIM3_CH1/PA6)
- new net Y-MIN: U?.21 (SPI1_SCK/DAC_OUT2/ADC12_IN5/PA5)
- new net Y-STEP: U?.61 (TIM4_CH3/SDIO_D4/PB8)
- new net Z-DIR: U?.10 (PC2/ADC123_IN12), U?.16 (DIR), U?.16 (DIR)
- new net Z-EN: U?.8 (PC0/ADC123_IN10), U?.9 (EN), U?.9 (EN)
- new net Z-MAX: U?.24 (PC4/ADC12_IN14)
- new net Z-MIN: U?.23 (SPI1_MOSI/TIM8_CH1N/ADC12_IN7/TIM3_CH2/PA7)
- new net Z-STEP: U?.15 (STEP), U?.15 (STEP), U?.9 (PC1/ADC123_IN11)

Commit message: KiCad Changes
Added some stuff
Parts:
- added P? (x2): CONN_01X04, symbol CONN_01X04
- added P?: CONN_01X05, symbol CONN_01X05
- added P? (x2): CONN_01X03, symbol CONN_01X03
- R? (x2): value R -> 100K
Connections:
- net +3V3: now also P?.1 (P1), P?.1 (P1), P?.1 (P1)
- net GND: now also P?.3 (P3), P?.3 (P3), P?.4 (P4), P?.4 (P4), P?.5 (P5)
- net NRST: now also P?.4 (P4)
- net SWCLK: now also P?.2 (P2)
- net SWDIO: now also P?.3 (P3)
- net UART1-RX: now also P?.3 (P3)
- net UART1-TX: now also P?.2 (P2)
- net BL-RX renamed UART2-RX
- net UART2-RX: now also P?.3 (P3)
- net BL-TX renamed UART2-TX
- net UART2-TX: now also P?.2 (P2)
- new net +5V: P?.1 (P1), P?.1 (P1)
- new net SERVO0,: P?.2 (P2)
- new net SRVO1: P?.2 (P2)
